File: hardware/openbook.sch (EAGLE design)
At the start: 103 parts, among them IC1 XC6220A331MR-G, IC2 BD5229G-TR, J1 SAMACSYS_PARTS_USB4110-GF-A, J2 112A-TAAR-R03_ATTEND, J3 QWIIC_RIGHT_ANGLE, J4 FH34SRJ-24S-0.5SH_99_, Q1 20V/4.2A/52mΩ/1.4W, Q2 20V/4.2A/52mΩ/1.4W, Q3 20V/4.2A/52mΩ/1.4W, U1 ESP32-C6-WROOM-1-N8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

Commit message: Fixed schematic issues
Changed lines of the file:
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@@
 </classes>
 <parts>
-<part name="FRAME1" library="Frames" library_urn="urn:adsk.eagle:library:42976481" deviceset="A3L-LOC" device=""/>
+<part name="FRAME1" library="Frames" library_urn="urn:adsk.eagle:library:42976481" deviceset="A3L-LOC" device="" value="openbook"/>
 <part name="J1" library="DeskAssistant v19 v1" library_urn="urn:adsk.wipprod:fs.file:vf.L-M1R32STL6kAumfhKZWqw" deviceset="SAMACSYS_PARTS_USB4110-GF-A" device=""/>
 <part name="GND1" library="DeskAssistant v19 v1" library_urn="urn:adsk.wipprod:fs.file:vf.L-M1R32STL6kAumfhKZWqw" deviceset="GND" device=""/>
@@
 <segment>
 <wire x1="149.86" y1="165.1" x2="142.24" y2="165.1" width="0.1524" layer="91"/>
-<wire x1="142.24" y1="165.1" x2="134.62" y2="165.1" width="0.1524" layer="91"/>
-<wire x1="142.24" y1="172.72" x2="142.24" y2="165.1" width="0.1524" layer="91"/>
-<junction x="142.24" y="165.1"/>
 <label x="142.24" y="170.18" size="1.016" layer="95" rot="R90" xref="yes"/>
 <pinref part="C15" gate="G$1" pin="2"/>
 <pinref part="J4" gate="G$1" pin="23"/>
+<wire x1="142.24" y1="165.1" x2="134.62" y2="165.1" width="0.1524" layer="91"/>
+<junction x="142.24" y="165.1"/>
+<wire x1="142.24" y1="165.1" x2="142.24" y2="170.18" width="0.1524" layer="91"/>
 </segment>
 </net>
@@
 </segment>
 <segment>
-<wire x1="149.86" y1="160.02" x2="134.62" y2="160.02" width="0.1524" layer="91"/>
-<wire x1="134.62" y1="160.02" x2="129.54" y2="160.02" width="0.1524" layer="91"/>
-<wire x1="134.62" y1="172.72" x2="134.62" y2="160.02" width="0.1524" layer="91"/>
-<junction x="134.62" y="160.02"/>
+<wire x1="149.86" y1="160.02" x2="137.16" y2="160.02" width="0.1524" layer="91"/>
 <label x="134.62" y="170.18" size="1.016" layer="95" rot="R90" xref="yes"/>
 <pinref part="C16" gate="G$1" pin="2"/>
 <pinref part="J4" gate="G$1" pin="21"/>
-</segment>
-</net>
+<wire x1="137.16" y1="160.02" x2="129.54" y2="160.02" width="0.1524" layer="91"/>
+<junction x="137.16" y="160.02"/>
+<wire x1="137.16" y1="160.02" x2="137.16" y2="170.18" width="0.1524" layer="91"/>
+<wire x1="137.16" y1="170.18" x2="134.62" y2="170.18" width="0.1524" layer="91"/>
+</segment>
+</net>
